File: LevelConverter.kicad_sch (KiCad schematic)
At the start: 6 parts, among them U3 MAX3232

Commit message: rev 1 DFM fixes, kibot automation
Parts:
- U3: footprint Package_SO:SOIC-16_3.9x9.9mm_P1.27mm -> Package_SO:TSSOP-16_4.4x5mm_P0.65mm
Changed lines of the file:
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@@
     (property "Reference" "U3" (id 0) (at 128.27 74.93 0))
     (property "Value" "MAX3232" (id 1) (at 128.27 77.47 0))
-    (property "Footprint" "Package_SO:SOIC-16_3.9x9.9mm_P1.27mm" (id 2) (at 129.54 111.76 0)
+    (property "Footprint" "Package_SO:TSSOP-16_4.4x5mm_P0.65mm" (id 2) (at 129.54 111.76 0)
       (effects (font (size 1.27 1.27)) (justify left) hide)
     )
