File: gpsdo-connector.kicad_sch (KiCad schematic)
At the start: 22 parts, among them J1 DC-005A-2.5A-2.0, J2 SQ_OUT, J3 SINE_OUT, J4 GPS_ACT, J5 MASTER, J6 FPC-50-0.5MM, P8 BeagleBone_Black_Header, P9 BeagleBone_Black_Header, U1 LM75B

Commit message: rev 1 DFM fixes, kibot automation
Parts:
- R1, R2, R3: LCSC (none) -> C17557
- R4: LCSC (none) -> C17414
- U1: LCSC (none) -> C2837470
Changed lines of the file:
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@@
+      (effects (font (size 1.27 1.27)) hide)
+    )
+    (property "LCSC" "C17557" (id 4) (at 85.09 148.59 0)
       (effects (font (size 1.27 1.27)) hide)
     )
@@
       (effects (font (size 1.27 1.27)) hide)
     )
+    (property "LCSC" "C2837470" (id 4) (at 144.78 156.21 0)
+      (effects (font (size 1.27 1.27)) hide)
+    )
     (pin "1")
     (pin "2")
@@
       (effects (font (size 1.27 1.27)) hide)
     )
+    (property "LCSC" "C17557" (id 4) (at 85.09 153.67 0)
+      (effects (font (size 1.27 1.27)) hide)
+    )
     (pin "1")
     (pin "2")
@@
     )
     (property "Datasheet" "~" (id 3) (at 26.67 148.59 0)
+      (effects (font (size 1.27 1.27)) hide)
+    )
+    (property "LCSC" "C17557" (id 4) (at 26.67 148.59 0)
       (effects (font (size 1.27 1.27)) hide)
     )
@@
     )
     (property "Datasheet" "~" (id 3) (at 195.58 73.66 0)
+      (effects (font (size 1.27 1.27)) hide)
+    )
+    (property "LCSC" "C17414" (id 4) (at 195.58 73.66 0)
       (effects (font (size 1.27 1.27)) hide)
     )
@@
     )
     (path "/00000000-0000-0000-0000-00005dc4d8af/00000000-0000-0000-0000-00005dc4dbe2"
-      (reference "U3") (unit 1) (value "MAX3232") (footprint "Package_SO:SOIC-16_3.9x9.9mm_P1.27mm")
+      (reference "U3") (unit 1) (value "MAX3232") (footprint "Package_SO:TSSOP-16_4.4x5mm_P0.65mm")
     )
     (path "/5d45b828-7e2f-48df-92fd-def32aa6a558/209f9bae-8fa6-4e41-9ad6-2ac835ee19ad/6f09f5d7-71b7-4ac5-98b6-6629dea616c4"
