File: power.kicad_sch (KiCad schematic)
At the start: 21 parts, among them U2 LMR14030SDDAR

Commit message: rev 1 DFM fixes, kibot automation
Parts:
- RV1: symbol gpsdo-connector-rescue:R_POT_TRIM-Device -> Device:R_Potentiometer_Trim
Changed lines of the file:
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@@
       (effects (font (size 1.27 1.27)) hide)
     )
-    (property "Datasheet" "" (id 3) (at 135.89 80.01 0)
+    (property "Datasheet" "https://www.ti.com/lit/ds/symlink/lmr14030.pdf" (id 3) (at 135.89 80.01 0)
       (effects (font (size 1.27 1.27)) hide)
     )
@@
       (effects (font (size 1.27 1.27)) hide)
     )
-    (property "Datasheet" "~" (id 3) (at 180.34 86.36 0)
+    (property "Datasheet" "http://www.pdc.com.tw/product/Power/Coil%E7%9B%AE%E9%8C%84%2083%20(POWER%20CHOKE%20(MOLDING)_MCS0630).pdf" (id 3) (at 180.34 86.36 0)
       (effects (font (size 1.27 1.27)) hide)
     )
@@
     (pin "2")
   )
-  (symbol (lib_id "gpsdo-connector-rescue:R_POT_TRIM-Device") (at 180.34 69.85 90) (unit 1)
+  (symbol (lib_id "Device:R_Potentiometer_Trim") (at 180.34 69.85 90) (unit 1)
     (in_bom yes) (on_board yes)
     (property "Reference" "RV1" (id 0) (at 180.34 62.23 90)
