File: rtc.kicad_sch (KiCad schematic)
At the start: 8 parts, among them U5 PCF8563T, Y1 32.768k

Commit message: rev 1 DFM fixes, kibot automation
Parts:
- R12, R13: LCSC (none) -> C4382
- U5: LCSC (none) -> C7440; MPN (none) -> PCF8563T/5,518
Changed lines of the file:
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@@
+      (effects (font (size 1.27 1.27)) hide)
+    )
+    (property "LCSC" "C4382" (id 4) (at 129.54 86.36 0)
       (effects (font (size 1.27 1.27)) hide)
     )
@@
       (effects (font (size 1.27 1.27)) hide)
     )
-    (property "Datasheet" "https://assets.nexperia.com/documents/data-sheet/PCF8563.pdf" (id 3) (at 109.22 96.52 0)
+    (property "Datasheet" "https://www.nxp.com/docs/en/data-sheet/PCF8563.pdf" (id 3) (at 109.22 96.52 0)
+      (effects (font (size 1.27 1.27)) hide)
+    )
+    (property "LCSC" "C7440" (id 4) (at 109.22 96.52 0)
+      (effects (font (size 1.27 1.27)) hide)
+    )
+    (property "MPN" "PCF8563T/5,518" (id 5) (at 109.22 96.52 0)
       (effects (font (size 1.27 1.27)) hide)
     )
@@
       (effects (font (size 1.27 1.27)) hide)
     )
+    (property "LCSC" "C4382" (id 4) (at 121.92 86.36 0)
+      (effects (font (size 1.27 1.27)) hide)
+    )
